File: RF Controller V-Final.kicad_sch (KiCad schematic)
At the start: 37 parts, among them J2 J_OLED, J3 BAT+, J4 BAT-, SW1 EG1218, U1 Teensy4.0, U3 NRF24L01, U5 AP2112K-3.3, U7 Pitch/Roll, U8 TPS542025DDCR, U9 Throttle/Yaw

Commit message: Component layout V1
Parts:
- C11: value 22u -> 10u
- C12: value 10u -> 22u
Connections:
- net 3.3V_OUT: now also C11.1; no longer C12.1
- net 5V_IN: now also C12.1; no longer C11.1
- net VBAT: now also SW1.1 (A); no longer SW1.3 (C)
- net BUCK_SW: now reaches C10.1, L1.1, U8.2 (SW)
Other:
- moved on the sheet: C10, C11, C12, L1, R6, R7, U8

Commit message: Saved schematic
Parts:
- C2: footprint 865080543009:WCAP-ASLI_6.3X5.5_DXL_ -> Capacitor_SMD_Wurth:CP_Wurth_WCAP-ASLI-D6.3L5.5
Changed lines of the file:
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@@
 			)
 		)
-		(property "Footprint" "865080543009:WCAP-ASLI_6.3X5.5_DXL_"
+		(property "Footprint" "Capacitor_SMD_Wurth:CP_Wurth_WCAP-ASLI-D6.3L5.5"
 			(at 16.51 95.25 0)
 			(hide yes)

Commit message: Modified 3.3V_OUT nets
Connections:
- net 3.3V_OUT: no longer U1.16 (3V3)
- no-connect marks 35 -> 36
Changed lines of the file:
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@@
+	)
+	(no_connect
+		(at 36.83 156.21)
 	)
 	(no_connect
@@
 		(pts
 			(xy 213.36 80.01) (xy 212.09 80.01)
-		)
-		(stroke
-			(width 0)
-			(type default)
-		)
-	)
-	(wire
-		(pts
-			(xy 35.56 156.21) (xy 36.83 156.21)
 		)
 		(stroke
@@
 		(effects
 			(font
-				(size 1.27 1.27)
-			)
-			(justify right bottom)
-		)
-	)
-	(label "3.3V_OUT"
-		(at 35.56 156.21 180)
-		(effects
-			(font

Commit message: rewired joystick to 3v3
Connections:
- net 3.3V_OUT: no longer U7.2 (+5v), U9.2 (+5v)
- net 3v3: now reaches U1.16 (3V3)
- net 3v3: now also U7.2 (+5v), U9.2 (+5v)
- no-connect marks 36 -> 35
Changed lines of the file:
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@@
-	)
-	(no_connect
-		(at 36.83 156.21)
 	)
 	(no_connect
@@
 	(wire
 		(pts
+			(xy 35.56 156.21) (xy 36.83 156.21)
+		)
+		(stroke
+			(width 0)
+			(type default)
+		)
+	)
+	(wire
+		(pts
 			(xy 25.4 67.31) (xy 25.4 64.77)
 		)
@@
 		)
 	)
-	(label "3.3V_OUT"
-		(at 238.76 58.42 180)
-		(effects
-			(font
-				(size 1.27 1.27)
-			)
-			(justify right bottom)
-		)
-	)
 	(label "9V_IN"
 		(at 22.86 63.5 180)
@@
 		)
 	)
+	(label "3v3"
+		(at 237.49 92.71 180)
+		(effects
+			(font
+				(size 1.27 1.27)
+			)
+			(justify right bottom)
+		)
+	)
 	(label "ADC1"
 		(at 36.83 171.45 180)
@@
 	)
 	(label "3.3V_OUT"
-		(at 237.49 92.71 180)
-		(effects
-			(font
-				(size 1.27 1.27)
-			)
-			(justify right bottom)
-		)
-	)
-	(label "3.3V_OUT"
 		(at 180.34 63.5 180)
 		(effects
@@
 		)
 	)
+	(label "3v3"
+		(at 35.56 156.21 180)
+		(effects
+			(font
+				(size 1.27 1.27)
+			)
+			(justify right bottom)
+		)
+	)
 	(label "5V_IN"
 		(at 93.98 176.53 0)
@@
 		)
 	)
+	(label "3v3"
+		(at 238.76 58.42 180)
+		(effects
+			(font
+				(size 1.27 1.27)
+			)
+			(justify right bottom)
+		)
+	)

Commit message: Added PWR_FLAG
Other:
- moved on the sheet: D6, SW1
Changed lines of the file:
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@@
 	)
 	(junction
+		(at 54.61 24.13)
+		(diameter 0)
+		(color 0 0 0 0)
+	)
+	(junction
 		(at 22.86 72.39)
 		(diameter 0)
@@
 	)
 	(junction
+		(at 53.34 57.15)
+		(diameter 0)
+		(color 0 0 0 0)
+	)
+	(junction
 		(at 250.19 35.56)
 		(diameter 0)
@@
 	)
 	(no_connect
-		(at 43.18 33.02)
+		(at 38.1 34.29)
 	)
 	(no_connect
@@
 		)
 	)
+	(wire
+		(pts
+			(xy 55.88 24.13) (xy 54.61 24.13)
+		)
+		(stroke
+			(width 0)
+			(type default)
+		)
+	)
 	(polyline
 		(pts
@@
 	)
 	(label "SW_OUT"
-		(at 53.34 35.56 0)
+		(at 48.26 36.83 0)
 		(effects
 			(font
@@
 	)
 	(label "9V_IN"
-		(at 54.61 20.32 0)
+		(at 55.88 24.13 0)
 		(effects
 			(font
@@
 	)
 	(label "VBAT"
-		(at 43.18 38.1 180)
+		(at 38.1 39.37 180)
 		(effects
 			(font
@@
 	)
 	(label "SW_OUT"
-		(at 46.99 20.32 180)
+		(at 46.99 24.13 180)
 		(effects
 			(font
@@
 	(symbol
 		(lib_id "Device:D_Schottky")
-		(at 50.8 20.32 180)
+		(at 50.8 24.13 180)
 		(unit 1)
 		(body_style 1)
@@
 		(dnp no)
 		(property "Reference" "D6"
-			(at 50.8 17.526 0)
+			(at 50.8 21.336 0)
 			(show_name no)
 			(do_not_autoplace no)
@@
 		)
 		(property "Value" "SS14"
-			(at 50.8 24.13 0)
+			(at 50.8 27.94 0)
 			(show_name no)
 			(do_not_autoplace no)
@@
 		)
 		(property "Footprint" "Diode_SMD:D_SMA"
-			(at 50.8 15.875 0)
+			(at 50.8 19.685 0)
 			(hide yes)
 			(show_name no)
@@
 		)
 		(property "Datasheet" "https://www.diodes.com/assets/Datasheets/SS14.pdf"
-			(at 50.8 20.32 0)
+			(at 50.8 24.13 0)
 			(hide yes)
 			(show_name no)
@@
 		)
 		(property "Description" "40V 1A Schottky barrier rectifier, SMA"
-			(at 50.8 20.32 0)
+			(at 50.8 24.13 0)
 			(hide yes)
 			(show_name no)
@@
 		)
 		(property "Sim.Device" "D"
-			(at 50.8 20.32 0)
+			(at 50.8 24.13 0)
 			(hide yes)
 			(show_name no)
@@
 		)
 		(property "Sim.Pins" "1=K 2=A"
-			(at 50.8 20.32 0)
+			(at 50.8 24.13 0)
 			(hide yes)
 			(show_name no)
@@
 	)
 	(symbol
+		(lib_id "power:PWR_FLAG")
+		(at 53.34 57.15 270)
+		(unit 1)
+		(body_style 1)
+		(exclude_from_sim no)
+		(in_bom yes)
+		(on_board yes)
+		(in_pos_files yes)
+		(dnp no)
+		(fields_autoplaced yes)
+		(property "Reference" "#FLG02"
+			(at 55.245 57.15 0)
+			(hide yes)
+			(show_name no)
+			(do_not_autoplace no)
+			(effects
+				(font
+					(size 1.27 1.27)
+				)
+			)
+		)
+		(property "Value" "PWR_FLAG"
+			(at 57.15 57.1499 90)
+			(show_name no)
+			(do_not_autoplace no)
+			(effects
+				(font
+					(size 1.27 1.27)
+				)
+				(justify left)
+			)
+		)
+		(property "Footprint" ""
+			(at 53.34 57.15 0)
+			(hide yes)
+			(show_name no)
+			(do_not_autoplace no)
+			(effects
+				(font
+					(size 1.27 1.27)
+				)
+			)
+		)
+		(property "Datasheet" ""
+			(at 53.34 57.15 0)
+			(hide yes)
+			(show_name no)
+			(do_not_autoplace no)
+			(effects
+				(font
+					(size 1.27 1.27)
+				)
+			)
+		)
+		(property "Description" "Special symbol for telling ERC where power comes from"
+			(at 53.34 57.15 0)
+			(hide yes)
+			(show_name no)
+			(do_not_autoplace no)
+			(effects
+				(font
+					(size 1.27 1.27)
+				)
+			)
+		)
+		(pin "1"
+		)
+		(instances
+			(project "RF Controller V-Final"
+				(path "/20b51a64-697d-4081-9410-2d5c496e59fa"
+					(reference "#FLG02")
+					(unit 1)
+				)
+			)
+		)
+	)
+	(symbol
 		(lib_id "power:GND")
 		(at 199.39 97.79 0)
@@
 	)
 	(symbol
+		(lib_id "power:PWR_FLAG")
+		(at 54.61 24.13 0)
+		(unit 1)
+		(body_style 1)
+		(exclude_from_sim no)
+		(in_bom yes)
+		(on_board yes)
+		(in_pos_files yes)
+		(dnp no)
+		(fields_autoplaced yes)
+		(property "Reference" "#FLG01"
+			(at 54.61 22.225 0)
+			(hide yes)
+			(show_name no)
+			(do_not_autoplace no)
+			(effects
+				(font
+					(size 1.27 1.27)
+				)
+			)
+		)
+		(property "Value" "PWR_FLAG"
+			(at 54.61 19.05 0)
+			(show_name no)
+			(do_not_autoplace no)
+			(effects
+				(font
+					(size 1.27 1.27)
+				)
+			)
+		)
+		(property "Footprint" ""
+			(at 54.61 24.13 0)
+			(hide yes)
+			(show_name no)
+			(do_not_autoplace no)
+			(effects
+				(font
+					(size 1.27 1.27)
+				)
+			)
+		)
+		(property "Datasheet" ""
+			(at 54.61 24.13 0)
+			(hide yes)
+			(show_name no)
+			(do_not_autoplace no)
+			(effects
+				(font
+					(size 1.27 1.27)
+				)
+			)
+		)
+		(property "Description" "Special symbol for telling ERC where power comes from"
+			(at 54.61 24.13 0)
+			(hide yes)
+			(show_name no)
+			(do_not_autoplace no)
+			(effects
+				(font
+					(size 1.27 1.27)
+				)
+			)
+		)
+		(pin "1"
+		)
+		(instances
+			(project "RF Controller V-Final"
+				(path "/20b51a64-697d-4081-9410-2d5c496e59fa"
+					(reference "#FLG01")
+					(unit 1)
+				)
+			)
+		)
+	)
+	(symbol
 		(lib_id "Mechanical:MountingHole")
 		(at 80.01 27.94 0)
@@
 	(symbol
 		(lib_id "Switch:SW_SPDT")
-		(at 48.26 35.56 180)
+		(at 43.18 36.83 180)
 		(unit 1)
 		(body_style 1)
@@
 		(dnp no)
 		(property "Reference" "SW1"
-			(at 47.498 27.178 0)
+			(at 42.418 28.448 0)
 			(show_name no)
 			(do_not_autoplace no)
@@
 		)
 		(property "Value" "EG1218"
-			(at 48.006 30.226 0)
+			(at 42.926 31.496 0)
 			(show_name no)
 			(do_not_autoplace no)
@@
 		)
 		(property "Footprint" "V2Power:SW_ES_EG1218"
-			(at 48.26 35.56 0)
+			(at 43.18 36.83 0)
 			(hide yes)
 			(show_name no)
@@
 		)
 		(property "Datasheet" "https://configured-product-images.s3.amazonaws.com/2D/specs/EG1218.pdf"
-			(at 48.26 35.56 0)
+			(at 43.18 36.83 0)
 			(hide yes)
 			(show_name no)
@@
 		)
 		(property "Description" "E-Switch EG1218 compact SPDT slide switch, 200mA at 30VDC; pin 1 is BAT+, pin 2 (COM) is BAT_SW, and pin 3 is explicitly unused"
-			(at 48.26 35.56 0)
+			(at 43.18 36.83 0)
 			(hide yes)
 			(show_name no)

Commit message: Modified voltage reg cap and res values
Parts:
- C7: value 10u -> 22u
- R6: value 71.5k -> 47k
- R7: value 20k -> 22k
Changed lines of the file:
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@@
 			)
 		)
-		(property "Value" "10u"
+		(property "Value" "22u"
 			(at 35.052 95.504 0)
 			(show_name no)
@@
 			)
 		)
-		(property "Value" "71.5k"
+		(property "Value" "47k"
 			(at 18.796 67.564 0)
 			(show_name no)
@@
 			)
 		)
-		(property "Value" "20k"
+		(property "Value" "22k"
 			(at 21.336 74.93 0)
 			(show_name no)

Commit message: Modified traces
Connections:
- net VBAT: now also SW1.3 (C); no longer SW1.1 (A)
Other:
- moved on the sheet: SW1
Changed lines of the file:
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@@
 	)
 	(no_connect
+		(at 40.64 39.37)
+	)
+	(no_connect
 		(at 36.83 123.19)
 	)
@@
 	)
 	(no_connect
-		(at 38.1 34.29)
-	)
-	(no_connect
 		(at 92.71 123.19)
 	)
@@
 	)
 	(label "SW_OUT"
-		(at 48.26 36.83 0)
+		(at 50.8 36.83 0)
 		(effects
 			(font
@@
 		)
 	)
-	(label "VBAT"
-		(at 38.1 39.37 180)
-		(effects
-			(font
-				(size 1.27 1.27)
-			)
-			(justify right bottom)
-		)
-	)
 	(label "3.3V_OUT"
 		(at 228.6 29.21 180)
@@
 		)
 	)
+	(label "VBAT"
+		(at 40.64 34.29 180)
+		(effects
+			(font
+				(size 1.27 1.27)
+			)
+			(justify right bottom)
+		)
+	)
 	(symbol
 		(lib_id "JOYY:_1")
@@
 	(symbol
 		(lib_id "Switch:SW_SPDT")
-		(at 43.18 36.83 180)
+		(at 45.72 36.83 180)
 		(unit 1)
 		(body_style 1)
@@
 		(dnp no)
 		(property "Reference" "SW1"
-			(at 42.418 28.448 0)
+			(at 44.958 29.464 0)
 			(show_name no)
 			(do_not_autoplace no)
@@
 		)
 		(property "Value" "EG1218"
-			(at 42.926 31.496 0)
+			(at 45.466 31.496 0)
 			(show_name no)
 			(do_not_autoplace no)
@@
 		)
 		(property "Footprint" "V2Power:SW_ES_EG1218"
-			(at 43.18 36.83 0)
+			(at 45.72 36.83 0)
 			(hide yes)
 			(show_name no)
@@
 		)
 		(property "Datasheet" "https://configured-product-images.s3.amazonaws.com/2D/specs/EG1218.pdf"
-			(at 43.18 36.83 0)
+			(at 45.72 36.83 0)
 			(hide yes)
 			(show_name no)
@@
 		)
 		(property "Description" "E-Switch EG1218 compact SPDT slide switch, 200mA at 30VDC; pin 1 is BAT+, pin 2 (COM) is BAT_SW, and pin 3 is explicitly unused"
-			(at 43.18 36.83 0)
+			(at 45.72 36.83 0)
 			(hide yes)
 			(show_name no)

Commit message: Edited resistor values
Parts:
- R4: value 27k -> 120k
- R5: value 10k -> 33k
Changed lines of the file:
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@@
 			)
 		)
-		(property "Value" "27k"
+		(property "Value" "120k"
 			(at 123.444 85.09 0)
 			(show_name no)
@@
 			)
 		)
-		(property "Value" "10k"
+		(property "Value" "33k"
 			(at 119.888 91.694 0)
 			(show_name no)
